File: keefighter.kicad_pcb (KiCad board)
At the start: 2 copper layers, 290 x 105 mm, 69 parts, among them SW0 SW_PUSH, SW1 SW_PUSH, SW10 SW_PUSH, SW11 SW_PUSH, SW12 SW_PUSH, SW13 SW_PUSH, SW14 SW_PUSH, SW15 SW_PUSH, SW16 SW_PUSH, SW17 SW_PUSH, SW2 SW_PUSH, SW3 SW_PUSH, SW4 SW_PUSH, SW5 SW_PUSH, SW6 SW_PUSH, SW7 SW_PUSH, SW8 SW_PUSH, SW9 SW_PUSH, U1 ProMicro

Commit message: Initial Commit
Parts:
- removed D0, D1, D10, D11, D12, D13, D14, D15, D16, D17, D2, D3, D4, D5, D6, D7, D8, D9: 1N4148, kbd:D3_TH_SMD_v2
- removed LED0, LED1, LED10, LED11, LED2, LED3, LED4, LED5, LED6, LED7, LED8, LED9: SK6812MINI, kbd:YS-SK6812MINI-E
- removed the REF** at (196.4, 82.6)
- removed the REF** at (103.0, 141.6)
- removed the REF** at (173.2, 154.3)
- removed the REF** at (146.4, 139.0)
- removed the REF** at (113.1, 138.4)
- removed the REF** at (137.1, 138.4)
- removed the REF** at (77.8, 173.9)
- removed the REF** at (347.8, 88.9)
- removed the REF** at (347.8, 173.9)
- removed the REF** at (77.8, 88.9)
- removed the REF** at (212.8, 88.9)
- removed the REF** at (212.8, 173.9)
- removed the REF** at (173.2, 167.3)
- removed the REF** at (124.1, 138.4)
- removed Ref** (x5): Val**, pro micro:PAD.03X.05
- removed Ref**: Val**, logo:logo
- removed SW0, SW1, SW2, SW3, SW4, SW5: SW_PUSH, Button_Switch_THT:SW_PUSH_6mm
- removed SW10, SW11, SW12, SW13, SW14, SW15, SW16, SW17, SW6, SW7, SW8, SW9: SW_PUSH, kbd:CherryMX_Hotswap
- removed U1: ProMicro, pro micro:SPARKFUN_PRO_MICRO
- added >NAME: >VALUE, lib:JOYSTICK, F.Cu at (88.7, 114.4)
- added >NAME: >VALUE, lib:JOYSTICK, F.Cu at (343.8, 142.4)
- added REF**: HRO-TYPE-C-31-M-12-HandSoldering, usbc:HRO-TYPE-C-31-M-12-HandSoldering, B.Cu at (91.9, 89.9)
- added REF**: SW_PUSH_6mm, Button_Switch_THT:SW_PUSH_6mm, F.Cu at (88.1, 146.0)
- added REF**: SW_PUSH_6mm, Button_Switch_THT:SW_PUSH_6mm, F.Cu at (80.3, 138.5)
- added REF**: SW_PUSH_6mm, Button_Switch_THT:SW_PUSH_6mm, F.Cu at (96.0, 138.5)
- added REF**: SW_PUSH_6mm, Button_Switch_THT:SW_PUSH_6mm, F.Cu at (88.1, 131.2)
- added REF**: Kailh_socket_PG1350_optional, lib:Kailh_socket_PG1350, F.Cu at (225.9, 145.5)
- added REF**: Kailh_socket_PG1350_optional, lib:Kailh_socket_PG1350, F.Cu at (278.9, 121.0)
- added REF**: Kailh_socket_PG1350_optional, lib:Kailh_socket_PG1350, F.Cu at (259.9, 123.6)
- added REF**: Kailh_socket_PG1350_optional, lib:Kailh_socket_PG1350, F.Cu at (242.2, 130.8)
- added REF**: Kailh_socket_PG1350_optional, lib:Kailh_socket_PG1350, F.Cu at (236.7, 170.9)
- added REF**: Kailh_socket_PG1350_optional, lib:Kailh_socket_PG1350, F.Cu at (313.3, 137.4)
- added REF**: SW_PUSH_6mm, Button_Switch_THT:SW_PUSH_6mm, F.Cu at (338.1, 117.6)
- added REF**: Kailh_socket_PG1350_optional, lib:Kailh_socket_PG1350, F.Cu at (253.3, 133.3)
- added REF**: Kailh_socket_PG1350_optional, lib:Kailh_socket_PG1350, F.Cu at (313.6, 110.2)
- added REF**: Kailh_socket_PG1350_optional, lib:Kailh_socket_PG1350, F.Cu at (256.3, 162.9)
- added REF**: Kailh_socket_PG1350_optional, lib:Kailh_socket_PG1350, F.Cu at (284.3, 132.5)
- added REF**: Kailh_socket_PG1350_optional, lib:Kailh_socket_PG1350, F.Cu at (284.5, 105.3)
- added REF**: Kailh_socket_PG1350_optional, lib:Kailh_socket_PG1350, F.Cu at (228.6, 118.2)
- added REF**: Kailh_socket_PG1350_optional, lib:Kailh_socket_PG1350, F.Cu at (254.9, 105.3)
- added REF**: Kailh_socket_PG1350_optional, lib:Kailh_socket_PG1350, F.Cu at (195.7, 170.9)
- added REF**: Kailh_socket_PG1350_optional, lib:Kailh_socket_PG1350, F.Cu at (216.2, 170.9)
- added REF**: Kailh_socket_PG1350_optional, lib:Kailh_socket_PG1350, F.Cu at (190.2, 130.8)
- added REF**: SW_PUSH_6mm, Button_Switch_THT:SW_PUSH_6mm, F.Cu at (353.7, 117.6)
- added REF**: Kailh_socket_PG1350_optional, lib:Kailh_socket_PG1350, F.Cu at (176.1, 162.9)
- added REF**: Kailh_socket_PG1350_optional, lib:Kailh_socket_PG1350, F.Cu at (172.5, 123.6)
- added REF**: Kailh_socket_PG1350_optional, lib:Kailh_socket_PG1350, F.Cu at (119.2, 137.4)
- added REF**: Kailh_socket_PG1350_optional, lib:Kailh_socket_PG1350, F.Cu at (206.5, 145.5)
- added REF**: Kailh_socket_PG1350_optional, lib:Kailh_socket_PG1350, F.Cu at (153.5, 121.0)
- added REF**: Kailh_socket_PG1350_optional, lib:Kailh_socket_PG1350, F.Cu at (203.8, 118.2)
- added REF**: Kailh_socket_PG1350_optional, lib:Kailh_socket_PG1350, F.Cu at (179.1, 133.3)
- added REF**: Kailh_socket_PG1350_optional, lib:Kailh_socket_PG1350, F.Cu at (148.0, 105.3)
- added REF**: Kailh_socket_PG1350_optional, lib:Kailh_socket_PG1350, F.Cu at (177.5, 105.3)
- added REF**: Kailh_socket_PG1350_optional, lib:Kailh_socket_PG1350, F.Cu at (118.8, 110.2)
- added REF**: SW_PUSH_6mm, Button_Switch_THT:SW_PUSH_6mm, F.Cu at (345.9, 125.0)
- added REF**: Kailh_socket_PG1350_optional, lib:Kailh_socket_PG1350, F.Cu at (148.1, 132.5)
- added REF**: SW_PUSH_6mm, Button_Switch_THT:SW_PUSH_6mm, F.Cu at (345.9, 110.2)
- added REF**: SW_PUSH_6mm, Button_Switch_THT:SW_PUSH_6mm, F.Cu at (326.5, 102.2)
- added REF**: SW_PUSH_6mm, Button_Switch_THT:SW_PUSH_6mm, F.Cu at (330.8, 164.7)
- added REF**: SW_PUSH_6mm, Button_Switch_THT:SW_PUSH_6mm, F.Cu at (97.1, 164.7)
- added REF**: SW_PUSH_6mm, Button_Switch_THT:SW_PUSH_6mm, F.Cu at (101.4, 102.2)
Routing:
- net vcc: track 488.3 -> 0.00 mm, vias 12 -> 0
- net col4: track 268.4 -> 0.00 mm, vias 4 -> 0
- net Net-(D13-Pad2): track 261.1 -> 0.00 mm, vias 2 -> 0
- net Net-(D12-Pad2): track 242.3 -> 0.00 mm, vias 2 -> 0
- net Net-(D11-Pad2): track 222.5 -> 0.00 mm, vias 2 -> 0
- net row0: track 197.6 -> 0.00 mm
- net row1: track 195.9 -> 0.00 mm
- net row2: track 194.4 -> 0.00 mm
- net Net-(D17-Pad2): track 193.7 -> 0.00 mm, vias 1 -> 0
- net col5: track 187.8 -> 0.00 mm, vias 6 -> 0
- net Net-(D10-Pad2): track 186.5 -> 0.00 mm
- net Net-(D6-Pad2): track 174.0 -> 0.00 mm, vias 2 -> 0
- net Net-(D9-Pad2): track 170.4 -> 0.00 mm, vias 2 -> 0
- net Net-(D16-Pad2): track 169.6 -> 0.00 mm, vias 2 -> 0
- net col0: track 161.5 -> 0.00 mm
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- removed copper zone on B.Cu, net gnd
- removed copper zone on F.Cu, net gnd
Other:
- board size 290 x 105 mm -> 285 x 96.6 mm
- rule pad_to_mask_clearance: 0.2 -> 0
- board text removed: "10"
- board text removed: "14"
- board text removed: "15"
- board text removed: "16"
- board text removed: "2"
- board text removed: "3"
- board text removed: "4"
- board text removed: "5"
- board text removed: "6"
- board text removed: "7"
- board text removed: "8"
- board text removed: "9"
- board text removed: "A0"
- board text removed: "A1"
- board text removed: "A2"
- board text removed: "A3"
- board text removed: "GND"
- board text removed: "JLCJLCJLCJLC"
- board text removed: "Keefighter Prototype by lulzsun"
- board text removed: "RAW"
- board text removed: "RST"
- board text removed: "RX1"
- board text removed: "TX0"
- board text removed: "VCC"

Commit message: asdfasf
Parts:
- removed >NAME: >VALUE, lib:JOYSTICK
- removed REF** (x11): SW_PUSH_6mm, Button_Switch_THT:SW_PUSH_6mm
- removed REF** (x23): Kailh_socket_PG1350_optional, lib:Kailh_socket_PG1350
- added C0: 0.1u, Capacitor_SMD:C_0805_2012Metric_Pad1.18x1.45mm_HandSolder, B.Cu at (150.2, 170.4)
- added C1: 0.1u, Capacitor_SMD:C_0805_2012Metric_Pad1.18x1.45mm_HandSolder, B.Cu at (150.6, 161.4)
- added C2: 0.1u, Capacitor_SMD:C_0805_2012Metric_Pad1.18x1.45mm_HandSolder, B.Cu at (155.1, 167.4)
- added C3: 0.1u, Capacitor_SMD:C_0805_2012Metric_Pad1.18x1.45mm_HandSolder, B.Cu at (150.6, 164.4)
- added C4: 10u, Capacitor_SMD:C_0805_2012Metric_Pad1.18x1.45mm_HandSolder, B.Cu at (150.2, 167.4)
- added C5: 22p, Capacitor_SMD:C_0805_2012Metric_Pad1.18x1.45mm_HandSolder, B.Cu at (155.1, 170.4)
- added C6: 22p, Capacitor_SMD:C_0805_2012Metric_Pad1.18x1.45mm_HandSolder, B.Cu at (144.0, 156.5)
- added C7: 1u, Capacitor_SMD:C_0805_2012Metric_Pad1.18x1.45mm_HandSolder, B.Cu at (135.5, 156.0)
- added D0: D, lib:D3_TH_SMD_v2, B.Cu at (92.4, 131.5)
- added D1: D, lib:D3_TH_SMD_v2, B.Cu at (97.3, 114.4)
- added D10: D, lib:D3_TH_SMD_v2, B.Cu at (316.5, 120.9)
- added D11: D, lib:D3_TH_SMD_v2, B.Cu at (333.8, 98.9)
- added D12: D, lib:D3_TH_SMD_v2, B.Cu at (337.5, 109.7)
- added D13: D, lib:D3_TH_SMD_v2, B.Cu at (84.6, 138.9)
- added D14: D, lib:D3_TH_SMD_v2, B.Cu at (85.3, 153.4)
- added D15: D, lib:D3_TH_SMD_v2, B.Cu at (93.2, 146.0)
- added D16: D, lib:D3_TH_SMD_v2, B.Cu at (116.3, 148.0)
- added D17: D, lib:D3_TH_SMD_v2, B.Cu at (145.3, 143.1)
- added D18: D, lib:D3_TH_SMD_v2, B.Cu at (176.3, 143.9)
- added D19: D, lib:D3_TH_SMD_v2, B.Cu at (203.7, 156.1)
- added D2: D, lib:D3_TH_SMD_v2, B.Cu at (108.7, 98.9)
- added D20: D, lib:D3_TH_SMD_v2, B.Cu at (228.7, 156.1)
- added D21: D, lib:D3_TH_SMD_v2, B.Cu at (256.1, 143.9)
- added D22: D, lib:D3_TH_SMD_v2, B.Cu at (287.1, 143.1)
- added D23: D, lib:D3_TH_SMD_v2, B.Cu at (316.1, 148.0)
- added D24: D, lib:D3_TH_SMD_v2, B.Cu at (345.3, 117.1)
- added D25: D, lib:D3_TH_SMD_v2, B.Cu at (345.3, 102.3)
- added D26: D, lib:D3_TH_SMD_v2, B.Cu at (94.3, 161.4)
- added D27: D, lib:D3_TH_SMD_v2, B.Cu at (173.3, 173.5)
- added D28: D, lib:D3_TH_SMD_v2, B.Cu at (190.2, 180.4)
- added D29: D, lib:D3_TH_SMD_v2, B.Cu at (216.2, 184.0)
- added D3: D, lib:D3_TH_SMD_v2, B.Cu at (116.0, 120.9)
- added D30: D, lib:D3_TH_SMD_v2, B.Cu at (242.2, 180.4)
- added D31: D, lib:D3_TH_SMD_v2, B.Cu at (259.1, 173.5)
- added D32: D, lib:D3_TH_SMD_v2, B.Cu at (338.1, 161.4)
- added D33: D, lib:D3_TH_SMD_v2, B.Cu at (352.4, 142.4)
- added D34: D, lib:D3_TH_SMD_v2, B.Cu at (353.2, 109.7)
- added D35: PRTR5V0U2X, lib:SOT143B, B.Cu at (92.5, 103.4)
- added D4: D, lib:D3_TH_SMD_v2, B.Cu at (150.8, 94.7)
- added D5: D, lib:D3_TH_SMD_v2, B.Cu at (180.4, 94.6)
- added D6: D, lib:D3_TH_SMD_v2, B.Cu at (206.7, 107.5)
- added D7: D, lib:D3_TH_SMD_v2, B.Cu at (225.8, 107.5)
- added D8: D, lib:D3_TH_SMD_v2, B.Cu at (252.1, 94.6)
- added D9: D, lib:D3_TH_SMD_v2, B.Cu at (281.6, 94.7)
- added F0: 500m, Fuse:Fuse_1206_3216Metric_Pad1.42x1.75mm_HandSolder, B.Cu at (103.5, 107.3)
- added J0: AVR-ISP-6, lib:Reset_Pretty-Mask, B.Cu at (105.1, 195.3)
- added JOY0: COM-09032, lib:XDCR_COM-09032, F.Cu at (88.7, 114.4)
- added R0: 10k, Resistor_SMD:R_0805_2012Metric_Pad1.20x1.40mm_HandSolder, B.Cu at (158.3, 158.6)
- added R1: 10k, Resistor_SMD:R_0805_2012Metric_Pad1.20x1.40mm_HandSolder, B.Cu at (153.5, 155.5)
- added R2: 22, Resistor_SMD:R_0805_2012Metric_Pad1.20x1.40mm_HandSolder, B.Cu at (121.4, 154.8)
- added R3: 22, Resistor_SMD:R_0805_2012Metric_Pad1.20x1.40mm_HandSolder, B.Cu at (121.4, 152.6)
- added R4: 5.1k, Resistor_SMD:R_0805_2012Metric_Pad1.20x1.40mm_HandSolder, B.Cu at (67.6, 112.9)
- added R5: 5.1k, Resistor_SMD:R_0805_2012Metric_Pad1.20x1.40mm_HandSolder, B.Cu at (63.1, 112.9)
- added SW10: SW_Push, lib:Kailh_socket_PG1350, F.Cu at (313.6, 110.2)
- added SW11: SW_Push, Button_Switch_THT:SW_PUSH_6mm, F.Cu at (326.5, 102.2)
- added SW12: SW_Push, Button_Switch_THT:SW_PUSH_6mm, F.Cu at (338.1, 117.6)
- added SW13: SW_Push, Button_Switch_THT:SW_PUSH_6mm, F.Cu at (80.3, 138.5)
- added SW14: SW_Push, Button_Switch_THT:SW_PUSH_6mm, F.Cu at (88.1, 146.0)
- added SW15: SW_Push, Button_Switch_THT:SW_PUSH_6mm, F.Cu at (96.0, 138.5)
- added SW16: SW_Push, lib:Kailh_socket_PG1350, F.Cu at (119.2, 137.4)
- added SW17: SW_Push, lib:Kailh_socket_PG1350, F.Cu at (148.1, 132.5)
- added SW17c: Kailh_socket_PG1350_optional, lib:Kailh_socket_PG1350, F.Cu at (153.5, 121.0)
- added SW18: SW_Push, lib:Kailh_socket_PG1350, F.Cu at (179.1, 133.3)
- added SW18c: Kailh_socket_PG1350_optional, lib:Kailh_socket_PG1350, F.Cu at (172.5, 123.6)
- added SW19: SW_Push, lib:Kailh_socket_PG1350, F.Cu at (206.5, 145.5)
- added SW19c: Kailh_socket_PG1350_optional, lib:Kailh_socket_PG1350, F.Cu at (190.2, 130.8)
- added SW2: SW_Push, Button_Switch_THT:SW_PUSH_6mm, F.Cu at (101.4, 102.2)
- added SW20c: Kailh_socket_PG1350_optional, lib:Kailh_socket_PG1350, F.Cu at (242.2, 130.8)
- added SW21: SW_Push, lib:Kailh_socket_PG1350, F.Cu at (253.3, 133.3)
- added SW21c: Kailh_socket_PG1350_optional, lib:Kailh_socket_PG1350, F.Cu at (259.9, 123.6)
- added SW22: SW_Push, lib:Kailh_socket_PG1350, F.Cu at (284.3, 132.5)
- added SW22c: Kailh_socket_PG1350_optional, lib:Kailh_socket_PG1350, F.Cu at (278.9, 121.0)
- added SW23: SW_Push, lib:Kailh_socket_PG1350, F.Cu at (313.3, 137.4)
- added SW24: SW_Push, Button_Switch_THT:SW_PUSH_6mm, F.Cu at (345.9, 125.0)
- added SW25: SW_Push, Button_Switch_THT:SW_PUSH_6mm, F.Cu at (345.9, 110.2)
- added SW26: SW_Push, Button_Switch_THT:SW_PUSH_6mm, F.Cu at (97.1, 164.7)
- added SW3: SW_Push, lib:Kailh_socket_PG1350, F.Cu at (118.8, 110.2)
- added SW30: SW_Push, lib:Kailh_socket_PG1350, F.Cu at (236.7, 170.9)
- added SW31: SW_Push, lib:Kailh_socket_PG1350, F.Cu at (256.3, 162.9)
- added SW32: SW_Push, Button_Switch_THT:SW_PUSH_6mm, F.Cu at (330.8, 164.7)
- added SW34: SW_Push, Button_Switch_THT:SW_PUSH_6mm, F.Cu at (353.7, 117.6)
- added SW35: SW_Push_Reset, Button_Switch_THT:SW_PUSH_6mm, B.Cu at (106.8, 140.8)
- added SW4: SW_Push, lib:Kailh_socket_PG1350, F.Cu at (148.0, 105.3)
- added SW5: SW_Push, lib:Kailh_socket_PG1350, F.Cu at (177.5, 105.3)
- added SW6: SW_Push, lib:Kailh_socket_PG1350, F.Cu at (203.8, 118.2)
- added SW7: SW_Push, lib:Kailh_socket_PG1350, F.Cu at (228.6, 118.2)
- added SW8: SW_Push, lib:Kailh_socket_PG1350, F.Cu at (254.9, 105.3)
- added SW9: SW_Push, lib:Kailh_socket_PG1350, F.Cu at (284.5, 105.3)
- added U0: ATmega32U4-AU, Package_QFP:TQFP-44_10x10mm_P0.8mm, B.Cu at (131.9, 166.0)
- added X0: XTAL, Crystal:Crystal_SMD_3225-4Pin_3.2x2.5mm_HandSoldering, B.Cu at (144.9, 160.9)
- JOY1: renamed from >NAME; value >VALUE -> COM-09032; footprint lib:JOYSTICK -> lib:XDCR_COM-09032
- SW0: renamed from REF**; value SW_PUSH_6mm -> SW_Push
- SW20, SW27, SW28, SW29: renamed from REF**; value Kailh_socket_PG1350_optional -> SW_Push
- USB0: renamed from REF**; value HRO-TYPE-C-31-M-12-HandSoldering -> HRO-TYPE-C-31-M-12
Connections:
- JOY1 pad B1A: (no net) -> col1
- JOY1 pad B2A: (no net) -> Net-(D33-Pad2)
- JOY1 pad H1: (no net) -> Net-(JOY1-PadH1)
- JOY1 pad H2: (no net) -> Net-(JOY1-PadH2)
- JOY1 pad H3: (no net) -> Net-(JOY1-PadH3)
- JOY1 pad V1: (no net) -> Net-(JOY1-PadV1)
- JOY1 pad V2: (no net) -> Net-(JOY1-PadV2)
- JOY1 pad V3: (no net) -> Net-(JOY1-PadV3)
- SW0 pad 1: (no net) -> Net-(D0-Pad2)
- SW0 pad 2: (no net) -> col0
- SW20 pad 1: (no net) -> Net-(D20-Pad2)
- SW20 pad 2: (no net) -> col1
- SW27 pad 1: (no net) -> Net-(D27-Pad2)
- SW27 pad 2: (no net) -> col1
- SW28 pad 1: (no net) -> Net-(D28-Pad2)
- SW28 pad 2: (no net) -> col1
- SW29 pad 1: (no net) -> Net-(D29-Pad2)
- SW29 pad 2: (no net) -> col1
- USB0 pad 1: (no net) -> GND
- USB0 pad 10: (no net) -> Net-(R4-Pad1)
- USB0 pad 11: (no net) -> VCC
- USB0 pad 12: (no net) -> GND
- USB0 pad 13: (no net) -> GND
- USB0 pad 2: (no net) -> VCC
- USB0 pad 3: (no net) -> Net-(USB0-Pad3)
- USB0 pad 4: (no net) -> Net-(R5-Pad2)
- USB0 pad 5: (no net) -> DN
- USB0 pad 6: (no net) -> DP
- USB0 pad 7: (no net) -> DN
- USB0 pad 8: (no net) -> DP
- USB0 pad 9: (no net) -> Net-(USB0-Pad9)
Routing:
- net DP: track 0.00 -> 74.6 mm
- net DN: track 0.00 -> 74.0 mm
- net D+: track 0.00 -> 13.5 mm
- net D-: track 0.00 -> 12.7 mm

Commit message: Use components/schematics from flatbox
jfedor2's flatbox will be used as a guide for building the Keefighter
Parts:
- removed C0, C1, C2, C3: 0.1u, Capacitor_SMD:C_0805_2012Metric_Pad1.18x1.45mm_HandSolder
- removed C4: 10u, Capacitor_SMD:C_0805_2012Metric_Pad1.18x1.45mm_HandSolder
- removed C5, C6: 22p, Capacitor_SMD:C_0805_2012Metric_Pad1.18x1.45mm_HandSolder
- removed C7: 1u, Capacitor_SMD:C_0805_2012Metric_Pad1.18x1.45mm_HandSolder
- removed D0, D1, D10, D11, D12, D13, D14, D15, D16, D17, D18, D19, D2, D20, D21, D22, D23, D24, D25, D26, D27, D28, D29, D3, D30, D31, D32, D33, D34, D4, D5, D6, D7, D8, D9: D, lib:D3_TH_SMD_v2
- removed D35: PRTR5V0U2X, lib:SOT143B
- removed F0: 500m, Fuse:Fuse_1206_3216Metric_Pad1.42x1.75mm_HandSolder
- removed J0: AVR-ISP-6, lib:Reset_Pretty-Mask
- removed R0, R1: 10k, Resistor_SMD:R_0805_2012Metric_Pad1.20x1.40mm_HandSolder
- removed R2, R3: 22, Resistor_SMD:R_0805_2012Metric_Pad1.20x1.40mm_HandSolder
- removed R4, R5: 5.1k, Resistor_SMD:R_0805_2012Metric_Pad1.20x1.40mm_HandSolder
- removed SW10, SW16, SW17, SW18, SW19, SW21, SW22, SW23, SW3, SW30, SW31, SW4, SW5, SW6, SW7, SW8, SW9: SW_Push, lib:Kailh_socket_PG1350
- removed SW11, SW12, SW13, SW14, SW15, SW2, SW24, SW25, SW26, SW32, SW34: SW_Push, Button_Switch_THT:SW_PUSH_6mm
- removed SW17c, SW18c, SW19c: Kailh_socket_PG1350_optional, lib:Kailh_socket_PG1350
- removed SW35: SW_Push_Reset, Button_Switch_THT:SW_PUSH_6mm
- removed U0: ATmega32U4-AU, Package_QFP:TQFP-44_10x10mm_P0.8mm
- removed X0: XTAL, Crystal:Crystal_SMD_3225-4Pin_3.2x2.5mm_HandSoldering
- added J1: Conn_02x02_Odd_Even, Connector_PinHeader_2.54mm:PinHeader_2x02_P2.54mm_Vertical, B.Cu at (102.9, 141.9)
- added J6: Conn_02x12_Odd_Even, Connector_PinHeader_2.54mm:PinHeader_2x12_P2.54mm_Vertical, F.Cu at (202.2, 101.6)
- added REF**: 60_Outline, lib:60_Outline-Modded, F.Cu at (216.2, 139.2)
- added SWL_0: B_START, Button_Switch_THT:SW_PUSH_6mm, F.Cu at (101.4, 102.2)
- added SWL_1: B_L1, lib:Kailh_socket_PG1350, F.Cu at (118.8, 110.2)
- added SWL_10: B_L8, lib:Kailh_socket_PG1350, F.Cu at (206.5, 145.5)
- added SWL_10c: Kailh_socket_PG1350_optional, lib:Kailh_socket_PG1350, F.Cu at (190.2, 130.8)
- added SWL_11: B_DPAD_L, Button_Switch_THT:SW_PUSH_6mm, F.Cu at (80.3, 138.5)
- added SWL_12: B_DPAD_D, Button_Switch_THT:SW_PUSH_6mm, F.Cu at (88.1, 146.0)
- added SWL_13: B_CAPTURE, Button_Switch_THT:SW_PUSH_6mm, F.Cu at (97.1, 164.7)
- added SWL_2: B_L2, lib:Kailh_socket_PG1350, F.Cu at (148.0, 105.3)
- added SWL_3: B_L3, lib:Kailh_socket_PG1350, F.Cu at (177.5, 105.3)
- added SWL_4: B_L4, lib:Kailh_socket_PG1350, F.Cu at (203.8, 118.2)
- added SWL_6: B_DPAD_R, Button_Switch_THT:SW_PUSH_6mm, F.Cu at (96.0, 138.5)
- added SWL_7: B_L5, lib:Kailh_socket_PG1350, F.Cu at (119.2, 137.4)
- added SWL_8: B_L6, lib:Kailh_socket_PG1350, F.Cu at (148.1, 132.5)
- added SWL_8c: Kailh_socket_PG1350_optional, lib:Kailh_socket_PG1350, F.Cu at (153.5, 121.0)
- added SWL_9: B_L7, lib:Kailh_socket_PG1350, F.Cu at (179.1, 133.3)
- added SWL_9c: Kailh_socket_PG1350_optional, lib:Kailh_socket_PG1350, F.Cu at (172.5, 123.6)
- added SWR_0: B_SELECT, Button_Switch_THT:SW_PUSH_6mm, F.Cu at (326.5, 102.2)
- added SWR_1: B_R1, lib:Kailh_socket_PG1350, F.Cu at (313.6, 110.2)
- added SWR_11: B_B, Button_Switch_THT:SW_PUSH_6mm, F.Cu at (345.9, 125.0)
- added SWR_12: B_Y, Button_Switch_THT:SW_PUSH_6mm, F.Cu at (338.1, 117.6)
- added SWR_13: B_HOME, Button_Switch_THT:SW_PUSH_6mm, F.Cu at (330.8, 164.7)
- added SWR_14: B_R9, lib:Kailh_socket_PG1350, F.Cu at (256.3, 162.9)
- added SWR_15: B_R10, lib:Kailh_socket_PG1350, F.Cu at (236.7, 170.9)
- added SWR_2: B_R2, lib:Kailh_socket_PG1350, F.Cu at (284.5, 105.3)
- added SWR_3: B_R3, lib:Kailh_socket_PG1350, F.Cu at (254.9, 105.3)
- added SWR_4: B_R4, lib:Kailh_socket_PG1350, F.Cu at (228.6, 118.2)
- added SWR_5: B_A, Button_Switch_THT:SW_PUSH_6mm, F.Cu at (353.7, 117.6)
- added SWR_6: B_X, Button_Switch_THT:SW_PUSH_6mm, F.Cu at (345.9, 110.2)
- added SWR_7: B_R5, lib:Kailh_socket_PG1350, F.Cu at (313.3, 137.4)
- added SWR_8: B_R6, lib:Kailh_socket_PG1350, F.Cu at (284.3, 132.5)
- added SWR_9: B_R7, lib:Kailh_socket_PG1350, F.Cu at (253.3, 133.3)
- SWL_14: renamed from SW27; value SW_Push -> B_L9
- SWL_15: renamed from SW28; value SW_Push -> B_L10
- SWL_5: renamed from SW0; value SW_Push -> B_DPAD_U
- SWM_0: renamed from SW29; value SW_Push -> B_JUMP
- SWR_10: renamed from SW20; value SW_Push -> B_R8
- turned SWR_10 to 15 degrees
- renumbered USB0 to J4
Connections:
- net DN renamed D_N
- net DP renamed D_P
- net Net-(JOY0-PadH2) renamed JOY_LX
- net Net-(JOY0-PadV2) renamed JOY_LY
- net Net-(JOY1-PadH2) renamed JOY_RX
- net Net-(JOY1-PadV2) renamed JOY_RY
- J4 pad 11: VCC -> +5V
- J4 pad 2: VCC -> +5V
- JOY0 pad B1A: col1 -> B_LCLICK
- JOY0 pad B2A: Net-(D1-Pad2) -> GND
- JOY0 pad H1: Net-(JOY0-PadH1) -> +5V
- JOY0 pad H3: Net-(JOY0-PadH3) -> GND
- JOY0 pad S1: Net-(JOY0-PadS1) -> GND
- JOY0 pad S2: Net-(JOY0-PadS1) -> GND
- JOY0 pad S4: Net-(JOY0-PadS1) -> GND
- JOY0 pad V1: Net-(JOY0-PadV1) -> +5V
- JOY0 pad V3: Net-(JOY0-PadV3) -> GND
- JOY1 pad B1A: col1 -> B_RCLICK
- JOY1 pad B2A: Net-(D33-Pad2) -> GND
- JOY1 pad H1: Net-(JOY1-PadH1) -> +5V
- JOY1 pad H3: Net-(JOY1-PadH3) -> GND
- JOY1 pad S1: Net-(JOY1-PadS1) -> GND
- JOY1 pad S2: Net-(JOY1-PadS1) -> GND
- JOY1 pad S3: Net-(JOY1-PadS1) -> GND
- JOY1 pad S4: Net-(JOY1-PadS1) -> GND
- JOY1 pad V1: Net-(JOY1-PadV1) -> +5V
- JOY1 pad V3: Net-(JOY1-PadV3) -> GND
- SWL_14 pad 1: Net-(D27-Pad2) -> B_L9
- SWL_14 pad 2: col1 -> GND
- SWL_15 pad 1: Net-(D28-Pad2) -> B_L10
- SWL_15 pad 2: col1 -> GND
- SWL_5 pad 1: Net-(D0-Pad2) -> B_DPAD_U
- SWL_5 pad 2: col0 -> GND
- SWM_0 pad 1: Net-(D29-Pad2) -> GND
- SWM_0 pad 2: col1 -> B_JUMP
- SWR_10 pad 1: Net-(D20-Pad2) -> GND
- SWR_10 pad 2: col1 -> B_R8
Routing:
- net D_P: track 74.6 -> 0.00 mm
- net D_N: track 74.0 -> 0.00 mm
- net D+: track 13.5 -> 0.00 mm
- net D-: track 12.7 -> 0.00 mm
Other:
- board size 285 x 96.6 mm -> 285 x 95.1 mm
