File: keefighter.kicad_pcb (KiCad board)
At the start: 2 copper layers, 285 x 95.1 mm, 45 parts, among them J1 Conn_02x02_Odd_Even, J4 HRO-TYPE-C-31-M-12, J6 Conn_02x12_Odd_Even, SW20c Kailh_socket_PG1350_optional, SW21c Kailh_socket_PG1350_optional, SW22c Kailh_socket_PG1350_optional

Commit message: JLCPCB ready for prod
Parts:
- removed J4: HRO-TYPE-C-31-M-12, usbc:HRO-TYPE-C-31-M-12-HandSoldering
- removed J6: Conn_02x12_Odd_Even, Connector_PinHeader_2.54mm:PinHeader_2x12_P2.54mm_Vertical
- removed JOY0, JOY1: COM-09032, lib:XDCR_COM-09032
- removed SW20c, SW21c, SW22c, SWL_10c, SWL_8c, SWL_9c: Kailh_socket_PG1350_optional, lib:Kailh_socket_PG1350
- removed SWL_0: B_START, Button_Switch_THT:SW_PUSH_6mm
- removed SWL_1: B_L1, lib:Kailh_socket_PG1350
- removed SWL_10: B_L8, lib:Kailh_socket_PG1350
- removed SWL_11: B_DPAD_L, Button_Switch_THT:SW_PUSH_6mm
- removed SWL_12: B_DPAD_D, Button_Switch_THT:SW_PUSH_6mm
- removed SWL_13: B_CAPTURE, Button_Switch_THT:SW_PUSH_6mm
- removed SWL_2: B_L2, lib:Kailh_socket_PG1350
- removed SWL_3: B_L3, lib:Kailh_socket_PG1350
- removed SWL_4: B_L4, lib:Kailh_socket_PG1350
- removed SWL_5: B_DPAD_U, Button_Switch_THT:SW_PUSH_6mm
- removed SWL_6: B_DPAD_R, Button_Switch_THT:SW_PUSH_6mm
- removed SWL_7: B_L5, lib:Kailh_socket_PG1350
- removed SWL_8: B_L6, lib:Kailh_socket_PG1350
- removed SWL_9: B_L7, lib:Kailh_socket_PG1350
- removed SWR_0: B_SELECT, Button_Switch_THT:SW_PUSH_6mm
- removed SWR_1: B_R1, lib:Kailh_socket_PG1350
- removed SWR_11: B_B, Button_Switch_THT:SW_PUSH_6mm
- removed SWR_12: B_Y, Button_Switch_THT:SW_PUSH_6mm
- removed SWR_13: B_HOME, Button_Switch_THT:SW_PUSH_6mm
- removed SWR_14: B_R9, lib:Kailh_socket_PG1350
- removed SWR_15: B_R10, lib:Kailh_socket_PG1350
- removed SWR_2: B_R2, lib:Kailh_socket_PG1350
- removed SWR_3: B_R3, lib:Kailh_socket_PG1350
- removed SWR_4: B_R4, lib:Kailh_socket_PG1350
- removed SWR_5: B_A, Button_Switch_THT:SW_PUSH_6mm
- removed SWR_6: B_X, Button_Switch_THT:SW_PUSH_6mm
- removed SWR_7: B_R5, lib:Kailh_socket_PG1350
- removed SWR_8: B_R6, lib:Kailh_socket_PG1350
- removed SWR_9: B_R7, lib:Kailh_socket_PG1350
- added C1: 1u, Capacitor_SMD:C_0603_1608Metric, B.Cu at (97.2, 111.6)
- added C10: 1u, Capacitor_SMD:C_0603_1608Metric, B.Cu at (203.2, 132.0)
- added C11: 100n, Capacitor_SMD:C_0603_1608Metric, B.Cu at (215.0, 136.0)
- added C12: 100n, Capacitor_SMD:C_0603_1608Metric, B.Cu at (201.2, 140.6)
- added C13: 100n, Capacitor_SMD:C_0603_1608Metric, B.Cu at (215.8, 140.6)
- added C14: 100n, Capacitor_SMD:C_0603_1608Metric, B.Cu at (207.4, 148.6)
- added C15: 100n, Capacitor_SMD:C_0603_1608Metric, B.Cu at (202.4, 136.0)
- added C16: 100n, Capacitor_SMD:C_0603_1608Metric, B.Cu at (202.4, 134.4)
- added C2: 30p, Capacitor_SMD:C_0603_1608Metric, B.Cu at (211.8, 151.0)
- added C3: 30p, Capacitor_SMD:C_0603_1608Metric, B.Cu at (207.4, 151.8)
- added C4: 1u, Capacitor_SMD:C_0603_1608Metric, B.Cu at (97.2, 105.6)
- added C5: 100n, Capacitor_SMD:C_0603_1608Metric, B.Cu at (207.0, 120.2)
- added C6: 100n, Capacitor_SMD:C_0603_1608Metric, B.Cu at (211.2, 129.4)
- added C7: 100n, Capacitor_SMD:C_0603_1608Metric, B.Cu at (205.8, 148.6)
- added C8: 1u, Capacitor_SMD:C_0603_1608Metric, B.Cu at (204.8, 131.2)
- added C9: 100n, Capacitor_SMD:C_0603_1608Metric, B.Cu at (209.6, 131.2)
- added R1: 1k, Resistor_SMD:R_0603_1608Metric, B.Cu at (215.0, 134.4)
- added R2: 10k, Resistor_SMD:R_0603_1608Metric, B.Cu at (212.6, 120.2)
- added R3: 27, Resistor_SMD:R_0603_1608Metric, B.Cu at (208.0, 131.2)
- added R4: 27, Resistor_SMD:R_0603_1608Metric, B.Cu at (206.4, 131.2)
- added R5: 1k, Resistor_SMD:R_0603_1608Metric, B.Cu at (209.2, 150.2)
- added R6: 5.1k, Resistor_SMD:R_0603_1608Metric, B.Cu at (87.2, 107.4)
- added R7: 5.1k, Resistor_SMD:R_0603_1608Metric, B.Cu at (83.4, 106.6)
- added REF**: MountingHole_2.2mm_M2_Pad, MountingHole:MountingHole_2.2mm_M2_Pad, F.Cu at (182.4, 102.1)
- added REF**: MountingHole_2.2mm_M2_Pad, MountingHole:MountingHole_2.2mm_M2_Pad, F.Cu at (235.7, 102.1)
- added REF**: MountingHole_2.2mm_M2_Pad, MountingHole:MountingHole_2.2mm_M2_Pad, F.Cu at (291.1, 102.1)
- added REF**: MountingHole_2.2mm_M2_Pad, MountingHole:MountingHole_2.2mm_M2_Pad, F.Cu at (346.5, 102.1)
- added REF**: MountingHole_2.2mm_M2_Pad, MountingHole:MountingHole_2.2mm_M2_Pad, F.Cu at (346.5, 186.7)
- added REF**: MountingHole_2.2mm_M2_Pad, MountingHole:MountingHole_2.2mm_M2_Pad, F.Cu at (291.1, 186.7)
- added REF**: MountingHole_2.2mm_M2_Pad, MountingHole:MountingHole_2.2mm_M2_Pad, F.Cu at (235.7, 186.7)
- added REF**: MountingHole_2.2mm_M2_Pad, MountingHole:MountingHole_2.2mm_M2_Pad, F.Cu at (182.4, 186.7)
- added REF**: MountingHole_2.2mm_M2_Pad, MountingHole:MountingHole_2.2mm_M2_Pad, F.Cu at (126.9, 186.7)
- added REF**: MountingHole_2.2mm_M2_Pad, MountingHole:MountingHole_2.2mm_M2_Pad, F.Cu at (71.5, 186.7)
- added REF**: MountingHole_2.2mm_M2_Pad, MountingHole:MountingHole_2.2mm_M2_Pad, F.Cu at (71.5, 102.1)
- added REF**: MountingHole_2.2mm_M2_Pad, MountingHole:MountingHole_2.2mm_M2_Pad, F.Cu at (126.9, 102.1)
- added Ref**: Val**, extra:logo, B.Cu at (107.0, 175.4)
- added SW1: SW_Push, Kailh:Kailh_socket_PG1350, F.Cu at (82.1, 112.7)
- added SW10: SW_Push, Kailh:Kailh_socket_PG1350, F.Cu at (336.0, 112.7)
- added SW11: SW_Push, Kailh:Kailh_socket_PG1350, F.Cu at (82.1, 131.7)
- added SW12: SW_Push, Kailh:Kailh_socket_PG1350, F.Cu at (109.0, 142.6)
- added SW13: SW_Push, Kailh:Kailh_socket_PG1350, F.Cu at (137.9, 137.7)
- added SW14: SW_Push, Kailh:Kailh_socket_PG1350, F.Cu at (168.9, 138.5)
- added SW15: SW_Push, Kailh:Kailh_socket_PG1350, F.Cu at (196.3, 150.7)
- added SW17: SW_Push, Kailh:Kailh_socket_PG1350, F.Cu at (249.1, 138.5)
- added SW18: SW_Push, Kailh:Kailh_socket_PG1350, F.Cu at (280.1, 137.7)
- added SW19: SW_Push, Kailh:Kailh_socket_PG1350, F.Cu at (309.1, 142.6)
- added SW2: SW_Push, Kailh:Kailh_socket_PG1350, F.Cu at (108.6, 115.4)
- added SW20: SW_Push, Kailh:Kailh_socket_PG1350, F.Cu at (336.0, 131.7)
- added SW21: SW_Push, Kailh:Kailh_socket_PG1350, F.Cu at (82.1, 150.7)
- added SW25: SW_Push, Kailh:Kailh_socket_PG1350, F.Cu at (229.5, 176.1)
- added SW26: SW_Push, Kailh:Kailh_socket_PG1350, F.Cu at (249.1, 168.1)
- added SW27: SW_Push, Kailh:Kailh_socket_PG1350, F.Cu at (336.0, 150.7)
- added SW28: SW_Push, Button_Switch_SMD:SW_Push_SPST_NO_Alps_SKRK, B.Cu at (95.7, 145.3)
- added SW29: SW_SPDT, Button_Switch_SMD:SW_SPDT_PCM12, B.Cu at (95.8, 140.0)
- added SW3: SW_Push, Kailh:Kailh_socket_PG1350, F.Cu at (137.8, 110.5)
- added SW4: SW_Push, Kailh:Kailh_socket_PG1350, F.Cu at (167.3, 110.5)
- added SW5: SW_Push, Kailh:Kailh_socket_PG1350, F.Cu at (193.6, 123.4)
- added SW6: SW_Push, Kailh:Kailh_socket_PG1350, F.Cu at (224.4, 123.4)
- added SW7: SW_Push, Kailh:Kailh_socket_PG1350, F.Cu at (250.7, 110.5)
- added SW8: SW_Push, Kailh:Kailh_socket_PG1350, F.Cu at (280.3, 110.5)
- added SW9: SW_Push, Kailh:Kailh_socket_PG1350, F.Cu at (309.4, 115.4)
- added SWb13: SW_Push, Kailh:Kailh_socket_PG1350, F.Cu at (143.3, 126.2)
- added SWb14: SW_Push, Kailh:Kailh_socket_PG1350, F.Cu at (162.3, 128.8)
- added SWb15: SW_Push, Kailh:Kailh_socket_PG1350, F.Cu at (180.0, 136.0)
- added SWb16: SW_Push, Kailh:Kailh_socket_PG1350, F.Cu at (238.0, 136.0)
- added SWb17: SW_Push, Kailh:Kailh_socket_PG1350, F.Cu at (255.7, 128.8)
- added SWb18: SW_Push, Kailh:Kailh_socket_PG1350, F.Cu at (274.7, 126.2)
- added U1: TLV74333PDBVR, Package_TO_SOT_SMD:SOT-23-5, B.Cu at (96.8, 108.6)
- added U2: W25Q128JVS, Package_SO:SOIC-8_5.23x5.23mm_P1.27mm, B.Cu at (209.8, 124.4)
- added U3: RP2040, RP2040:RP2040-QFN-56, B.Cu at (209.0, 139.5)
- added USB1: HRO-TYPE-C-31-M-12, Type-C:HRO-TYPE-C-31-M-12-Assembly, B.Cu at (84.7, 95.1)
- added Y1: Crystal_GND24, Crystal:Crystal_SMD_3225-4Pin_3.2x2.5mm, B.Cu at (210.2, 154.0)
- J1: value Conn_02x02_Odd_Even -> Conn_02x15_Odd_Even; footprint Connector_PinHeader_2.54mm:PinHeader_2x02_P2.54mm_Vertical -> Connector_PinHeader_2.54mm:PinHeader_2x15_P2.54mm_Vertical; moved to F.Cu
- SW16: renamed from SWR_10; value B_R8 -> SW_Push; footprint lib:Kailh_socket_PG1350 -> Kailh:Kailh_socket_PG1350
- SW22: renamed from SWL_14; value B_L9 -> SW_Push; footprint lib:Kailh_socket_PG1350 -> Kailh:Kailh_socket_PG1350
- SW23: renamed from SWL_15; value B_L10 -> SW_Push; footprint lib:Kailh_socket_PG1350 -> Kailh:Kailh_socket_PG1350
- SW24: renamed from SWM_0; value B_JUMP -> SW_Push; footprint lib:Kailh_socket_PG1350 -> Kailh:Kailh_socket_PG1350
- moved J1 96.4 mm to (191.2, 103.4), turned to 90 degrees
- moved REF** 8.88 mm to (209.0, 144.4)
- moved SW23 8.88 mm to (188.5, 176.1)
- moved SW24 8.88 mm to (209.0, 176.1)
- moved SW22 8.88 mm to (168.9, 168.1)
- moved SW16 6.68 mm to (221.7, 150.7)
Connections:
- net BOOT renamed Net-(J1-Pad4)
- J1 pad 2: GND -> +5V
- J1 pad 3: RESET -> F5
- SW16 pad 2: B_R8 -> F13
- SW22 pad 1: B_L9 -> F17
- SW23 pad 1: B_L10 -> F18
- SW24 pad 1: GND -> F19
- SW24 pad 2: B_JUMP -> GND
Routing:
- net OPT6: track 0.00 -> 341.6 mm, vias 0 -> 2
- net OPT5: track 0.00 -> 305.6 mm, vias 0 -> 2
- net OPT3: track 0.00 -> 281.9 mm, vias 0 -> 3
- net OPT4: track 0.00 -> 278.5 mm, vias 0 -> 2
- net OPT2: track 0.00 -> 276.5 mm, vias 0 -> 1
- net OPT1: track 0.00 -> 266.3 mm, vias 0 -> 1
- net F12: track 0.00 -> 221.0 mm
- net +3V3: track 0.00 -> 216.5 mm
- net F5: track 0.00 -> 214.1 mm, vias 0 -> 3
- net F1: track 0.00 -> 211.1 mm, vias 0 -> 1
- net GND: track 0.00 -> 164.8 mm, vias 0 -> 24
- net F6: track 0.00 -> 162.0 mm, vias 0 -> 4
- net D+: track 0.00 -> 161.2 mm
- net F15: track 0.00 -> 160.6 mm, vias 0 -> 3
- net F11: track 0.00 -> 159.7 mm
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- added copper zone on B.Cu, net GND
Other:
- net class Default: trace_width 0.25 -> 0.2; via_dia 0.8 -> 0.6; via_drill 0.4 -> 0.35
- net class FatPower added: clearance 0.2, trace_width 0.4, via_dia 0.6, via_drill 0.35
- net class Power added: clearance 0.15, trace_width 0.2, via_dia 0.6, via_drill 0.35
- net class dPair added: clearance 0.2, trace_width 0.2, via_dia 0.8, via_drill 0.4
- board text added: "Keefighter Rev.2 https://github.com/lulzsun/Keefighter"
