File: keefighter.sch (KiCad schematic (older format))
At the start: 82 parts, among them J6 Conn_02x12_Odd_Even, SW1 SW_Push, SW10 SW_Push, SW11 SW_Push, SW12 SW_Push, SW13 SW_Push, SW14 SW_Push, SW15 SW_Push, SW16 SW_Push, SW17 SW_Push, SW18 SW_Push, SW19 SW_Push, SW2 SW_Push, SW20 SW_Push, SW3 SW_Push, SW4 SW_Push, SW5 SW_Push, SW6 SW_Push, SW7 SW_Push, SW8 SW_Push, SW9 SW_Push, U1 TLV73333PDBV, U2 W25Q128JVS, U3 RP2040, Y1 Crystal_GND24

Commit message: JLCPCB ready for prod
Parts:
- removed SW1, SW2, SW3, SW4, SW5, SW6: SW_Push, Button_Switch_THT:SW_PUSH_6mm_H5mm, symbol Switch:SW_Push
- removed SW10, SW11, SW12, SW13, SW14, SW15, SW16, SW17, SW18, SW7, SW8, SW9: SW_Push, Kailh:Kailh_socket_PG1350_optional, symbol Switch:SW_Push
- removed SWL_11: B_DPAD_L, symbol Switch:SW_Push
- removed SWL_13: B_CAPTURE, symbol Switch:SW_Push
- removed SWL_5: B_DPAD_U, symbol Switch:SW_Push
- removed SWR_11: B_B, symbol Switch:SW_Push
- removed SWR_13: B_HOME, symbol Switch:SW_Push
- removed SWR_5: B_A, symbol Switch:SW_Push
- added SWb13, SWb14, SWb15, SWb16, SWb17, SWb18: SW_Push, Kailh:Kailh_socket_PG1350, symbol Switch:SW_Push
- C1, C10, C4, C8: footprint Capacitor_SMD:C_0402_1005Metric -> Capacitor_SMD:C_0603_1608Metric; LCSC C52923 -> C15849
- C11, C12, C13, C14, C15, C16, C5, C6, C7, C9: footprint Capacitor_SMD:C_0402_1005Metric -> Capacitor_SMD:C_0603_1608Metric; LCSC C1525 -> C14663
- C2, C3: footprint Capacitor_SMD:C_0402_1005Metric -> Capacitor_SMD:C_0603_1608Metric; LCSC C1570 -> C22397
- J1: renamed from J6; value Conn_02x12_Odd_Even -> Conn_02x15_Odd_Even; footprint Connector_PinHeader_2.54mm:PinHeader_2x12_P2.54mm_Vertical -> Connector_PinHeader_2.54mm:PinHeader_2x15_P2.54mm_Vertical; symbol Connector_Generic:Conn_02x12_Odd_Even -> Connector_Generic:Conn_02x15_Odd_Even
- R1, R5: footprint Resistor_SMD:R_0402_1005Metric -> Resistor_SMD:R_0603_1608Metric; LCSC C11702 -> C21190
- R2: footprint Resistor_SMD:R_0402_1005Metric -> Resistor_SMD:R_0603_1608Metric; LCSC C25744 -> C25804
- R3, R4: footprint Resistor_SMD:R_0402_1005Metric -> Resistor_SMD:R_0603_1608Metric; LCSC C138021 -> C25190
- R6, R7: footprint Resistor_SMD:R_0402_1005Metric -> Resistor_SMD:R_0603_1608Metric; LCSC C25905 -> C23186
- SW1: renamed from SWL_0; value B_START -> SW_Push; footprint (none) -> Kailh:Kailh_socket_PG1350
- SW10: renamed from SWR_0; value B_SELECT -> SW_Push; footprint (none) -> Kailh:Kailh_socket_PG1350
- SW11: renamed from SWL_6; value B_DPAD_R -> SW_Push; footprint (none) -> Kailh:Kailh_socket_PG1350
- SW12: renamed from SWL_7; value B_L5 -> SW_Push; footprint (none) -> Kailh:Kailh_socket_PG1350
- SW13: renamed from SWL_8; value B_L6 -> SW_Push; footprint (none) -> Kailh:Kailh_socket_PG1350
- SW14: renamed from SWL_9; value B_L7 -> SW_Push; footprint (none) -> Kailh:Kailh_socket_PG1350
- SW15: renamed from SWL_10; value B_L8 -> SW_Push; footprint (none) -> Kailh:Kailh_socket_PG1350
- SW16: renamed from SWR_10; value B_R8 -> SW_Push; footprint (none) -> Kailh:Kailh_socket_PG1350
- SW17: renamed from SWR_9; value B_R7 -> SW_Push; footprint (none) -> Kailh:Kailh_socket_PG1350
- SW18: renamed from SWR_8; value B_R6 -> SW_Push; footprint (none) -> Kailh:Kailh_socket_PG1350
- SW19: renamed from SWR_7; value B_R5 -> SW_Push; footprint (none) -> Kailh:Kailh_socket_PG1350
- SW2: renamed from SWL_1; value B_L1 -> SW_Push; footprint (none) -> Kailh:Kailh_socket_PG1350
- SW20: renamed from SWR_6; value B_X -> SW_Push; footprint (none) -> Kailh:Kailh_socket_PG1350
- SW21: renamed from SWL_12; value B_DPAD_D -> SW_Push; footprint (none) -> Kailh:Kailh_socket_PG1350
- SW22: renamed from SWL_14; value B_L9 -> SW_Push; footprint (none) -> Kailh:Kailh_socket_PG1350
- SW23: renamed from SWL_15; value B_L10 -> SW_Push; footprint (none) -> Kailh:Kailh_socket_PG1350
- SW24: renamed from SWM_0; value B_JUMP -> SW_Push; footprint (none) -> Kailh:Kailh_socket_PG1350
- SW25: renamed from SWR_15; value B_R10 -> SW_Push; footprint (none) -> Kailh:Kailh_socket_PG1350
- SW26: renamed from SWR_14; value B_R9 -> SW_Push; footprint (none) -> Kailh:Kailh_socket_PG1350
- SW27: renamed from SWR_12; value B_Y -> SW_Push; footprint (none) -> Kailh:Kailh_socket_PG1350
- SW28: renamed from SW20; footprint Button_Switch_SMD:SW_SPST_Omron_B3FS-100xP -> Button_Switch_SMD:SW_Push_SPST_NO_Alps_SKRK; LCSC C271750 -> C115357
- SW29: renamed from SW19; value SW_Push -> SW_SPDT; footprint Button_Switch_SMD:SW_SPST_Omron_B3FS-100xP -> Button_Switch_SMD:SW_SPDT_PCM12; symbol Switch:SW_Push -> Switch:SW_SPDT; LCSC C271750 -> C431541
- SW3: renamed from SWL_2; value B_L2 -> SW_Push; footprint (none) -> Kailh:Kailh_socket_PG1350
- SW4: renamed from SWL_3; value B_L3 -> SW_Push; footprint (none) -> Kailh:Kailh_socket_PG1350
- SW5: renamed from SWL_4; value B_L4 -> SW_Push; footprint (none) -> Kailh:Kailh_socket_PG1350
- SW6: renamed from SWR_4; value B_R4 -> SW_Push; footprint (none) -> Kailh:Kailh_socket_PG1350
- SW7: renamed from SWR_3; value B_R3 -> SW_Push; footprint (none) -> Kailh:Kailh_socket_PG1350
- SW8: renamed from SWR_2; value B_R2 -> SW_Push; footprint (none) -> Kailh:Kailh_socket_PG1350
- SW9: renamed from SWR_1; value B_R1 -> SW_Push; footprint (none) -> Kailh:Kailh_socket_PG1350
- U1: value TLV73333PDBV -> TLV74333PDBVR; LCSC C134139 -> C408972
Connections:
- net B_DPAD_D is gone; now on net OPT3: SW21.1
- net B_DPAD_R is gone; now on net OPT2: SW11.1
- net B_R10 is gone; now on net GND: SW25.2
- net B_RX is gone; now on net OPT5: SW20.2
- net B_Y is gone; now on net OPT6: SW27.2
- net CIRCLE is gone; now on net OPT2: U3.36 (GPIO24)
- net CROSS is gone; now on net F5: U3.30 (GPIO19)
- net DOWN is gone; now on net F13: U3.13 (GPIO10)
- net L1 is gone; now on net F4: U3.41 (GPIO29_ADC3)
- net LEFT is gone; now on net F14: U3.12 (GPIO9)
- net R1 is gone; now on net F2: U3.39 (GPIO27_ADC1)
- net R2 is gone; now on net F1: U3.38 (GPIO26_ADC0)
- net TRIANGLE is gone; now on net OPT1: U3.37 (GPIO25)
- net UP is gone; now on net F18: U3.27 (GPIO16)
- net +5V: now also J1.2 (Pin_2); no longer J1.14 (Pin_14)
- net GND: now also J1.1 (Pin_1), SW24.2, SW26.2, SW29.2 (B), SWb13.2, SWb14.2, SWb15.2, SWb16.1, SWb17.1, SWb18.1; no longer J1.12 (Pin_12), SW24.1, SW25.1, SW26.1, SW29.1
- net OPT1: now also J1.16 (Pin_16), SW1.1; no longer U3.8 (GPIO6)
- net OPT2: now also J1.14 (Pin_14); no longer U3.7 (GPIO5)
- net OPT3: now also J1.12 (Pin_12), U3.35 (GPIO23); no longer U3.6 (GPIO4)
- net OPT4: now also J1.22 (Pin_22), SW10.2, U3.6 (GPIO4); no longer U3.5 (GPIO3)
- net OPT5: now also J1.20 (Pin_20), U3.7 (GPIO5); no longer U3.4 (GPIO2)
- net OPT6: now also J1.18 (Pin_18), U3.8 (GPIO6); no longer U3.3 (GPIO1)
- net F15: now reaches U3.11 (GPIO8)
- net F15: now also J1.27 (Pin_27), SW18.2, SWb18.2
- net F19: now reaches U3.15 (GPIO12)
- net F19: now also J1.17 (Pin_17), SW24.1
- net F20: now reaches U3.16 (GPIO13)
- net F20: now also J1.19 (Pin_19), SW25.1
- net F21: now reaches U3.17 (GPIO14)
- net F21: now also J1.21 (Pin_21), SW26.1
- net F9: now reaches U3.2 (GPIO0)
- net F9: now also J1.30 (Pin_30), SW6.2
- net F17: now reaches U3.28 (GPIO17)
- net F17: now also J1.13 (Pin_13), SW22.1
- net F6: now reaches U3.31 (GPIO20)
- net F6: now also J1.5 (Pin_5), SW13.1, SWb13.1
- net F7: now reaches U3.32 (GPIO21)
- net F7: now also J1.7 (Pin_7), SW14.1, SWb14.1
- net F8: now reaches U3.34 (GPIO22)
- net F8: now also J1.9 (Pin_9), SW15.1, SWb15.1
- net F16: now reaches U3.9 (GPIO7)
- net F16: now also J1.29 (Pin_29), SW19.2
- net at R1.2: now also SW29.3 (C); no longer SW29.2
- net F4: now reaches J1.11 (Pin_11)
- net F4: now also SW5.1
- removed net B_JUMP: J1.13 (Pin_13), SW24.2
- net B_L1 renamed F1
- net F1: now also J1.10 (Pin_10); no longer J1.8 (Pin_8)
- net B_L10 renamed F18
- net F18: now also J1.15 (Pin_15)
- net B_L2 renamed F2
- net F2: now also J1.8 (Pin_8); no longer J1.6 (Pin_6)
- net B_L3: no longer names the net of J1.4 (Pin_4)
- net B_L3: no longer SW4.1
- removed net B_L4: J1.2 (Pin_2), SW5.1
- net B_L5 renamed F5
- net F5: now also J1.3 (Pin_3); no longer J1.1 (Pin_1)
- removed net B_L6: J1.3 (Pin_3), SW13.1
- removed net B_L7: J1.5 (Pin_5), SW14.1
- removed net B_L8: J1.7 (Pin_7), SW15.1
- removed net B_L9: J1.9 (Pin_9), SW22.1
- net B_R1 renamed F12
- net F12: now also J1.24 (Pin_24), U3.5 (GPIO3); no longer J1.18 (Pin_18)
- net B_R2 renamed F11
- net F11: now also J1.26 (Pin_26), U3.4 (GPIO2); no longer J1.20 (Pin_20)
- net B_R3 renamed F10
- net F10: now also J1.28 (Pin_28), U3.3 (GPIO1); no longer J1.22 (Pin_22)
- removed net B_R4: J1.24 (Pin_24), SW6.2
- net B_R5 renamed F13
- net F13: now also SW16.2, SWb16.2; no longer SW19.2
- removed net B_R6: J1.21 (Pin_21), SW18.2
- net B_R7 renamed F14
- net F14: now also J1.25 (Pin_25), SWb17.2; no longer J1.19 (Pin_19)
- removed net B_R8: J1.17 (Pin_17), SW16.2
- removed net B_R9: J1.15 (Pin_15), SW26.2
- removed net B_SELECT: J1.16 (Pin_16), SW10.2
- removed net B_START: J1.10 (Pin_10), SW1.1
- net L2 renamed F3
- net F3: now also J1.6 (Pin_6), SW4.1
- net RIGHT: no longer names the net of U3.14 (GPIO11)
- net SQUARE: no longer names the net of U3.29 (GPIO18)
- no-connect marks 17 -> 9
Other:
- moved on the sheet: C1, C10, C11, C12, C13, C14, C15, C16, C2, C3, C4, C5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
